File: pcb/hexapod/hexapod.kicad_pcb (KiCad board)
At the start: 2 copper layers, 109.5 x 113.5 mm, 19 parts, among them J1 Conn_01x03, J10 Conn_01x03, J11 Conn_01x03, J12 Conn_01x03, J13 Conn_01x03, J14 Conn_01x03, J15 Conn_01x03, J16 Conn_01x03, J17 Conn_01x03, J18 Conn_01x03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

Commit message: update
Connections:
- U1 pad 1: /l1_j1 -> unconnected-(U1-GPIO0-Pad1)
- U1 pad 10: /l3_j2 -> /l1_j1
- U1 pad 11: /l3_j3 -> /l1_j2
- U1 pad 12: unconnected-(U1-GPIO9-Pad12) -> /l1_j3
- U1 pad 14: unconnected-(U1-GPIO10-Pad14) -> /l2_j1
- U1 pad 15: unconnected-(U1-GPIO11-Pad15) -> /l2_j2
- U1 pad 16: unconnected-(U1-GPIO12-Pad16) -> /l2_j3
- U1 pad 17: unconnected-(U1-GPIO13-Pad17) -> /l3_j1
- U1 pad 19: unconnected-(U1-GPIO14-Pad19) -> /l3_j2
- U1 pad 2: /l1_j2 -> unconnected-(U1-GPIO1-Pad2)
- U1 pad 20: unconnected-(U1-GPIO15-Pad20) -> /l3_j3
- U1 pad 4: /l1_j3 -> unconnected-(U1-GPIO2-Pad4)
- U1 pad 5: /l2_j1 -> unconnected-(U1-GPIO3-Pad5)
- U1 pad 6: /l2_j2 -> unconnected-(U1-GPIO4-Pad6)
- U1 pad 7: /l2_j3 -> unconnected-(U1-GPIO5-Pad7)
- U1 pad 9: /l3_j1 -> unconnected-(U1-GPIO6-Pad9)
Routing:
- net (no net): vias 2 -> 0

Commit message: pcb design
Parts:
- added D1: D_Schottky, Diode_THT:D_T-1_P10.16mm_Horizontal, F.Cu at (105.0, 70.5)
- added J19: Conn_01x02, TerminalBlock:TerminalBlock_MaiXu_MX126-5.0-02P_1x02_P5.00mm, F.Cu at (98.0, 50.8)
- added U2: ~, Hexapod_Library:Mini360, F.Cu at (89.0, 53.7)
- added U3: ~, Hexapod_Library:Mini360, F.Cu at (109.0, 140.5)
- added U4: ~, Hexapod_Library:Mini360, F.Cu at (77.0, 147.1)
- added U5: ~, Hexapod_Library:Mini360, F.Cu at (123.0, 53.7)
- added U6: ~, Hexapod_Library:Mini360, F.Cu at (90.8, 141.3)
- added U7: ~, Hexapod_Library:Mini360, F.Cu at (111.0, 147.1)
- added U8: ~, Hexapod_Library:Mini360, F.Cu at (109.0, 68.0)
- moved J10 81.1 mm to (116.2, 75.5)
- moved J11 80.8 mm to (116.2, 79.5)
- moved J12 80.3 mm to (116.2, 83.5)
- moved J13 76.1 mm to (116.2, 96.0)
- moved J14 75.3 mm to (116.2, 100.0)
- moved J15 74.2 mm to (116.2, 104.0)
- moved J16 73.7 mm to (116.2, 117.0)
- moved J18 73.0 mm to (116.2, 125.0)
- moved J17 73.0 mm to (116.2, 121.0)
- moved J1 37.8 mm to (83.8, 76.0)
- moved J4 36.5 mm to (83.8, 96.0)
- moved J2 36.2 mm to (83.8, 80.0)
- moved J3 35.4 mm to (83.8, 84.0)
- moved J5 33.8 mm to (83.8, 100.0)
- moved J6 32.0 mm to (83.8, 104.0)
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Connections:
- J1 pad 2: unconnected-(J1-Pin_2-Pad2) -> /power_l1
- J10 pad 2: unconnected-(J10-Pin_2-Pad2) -> /power_r1
- J11 pad 2: unconnected-(J11-Pin_2-Pad2) -> /power_r1
- J12 pad 2: unconnected-(J12-Pin_2-Pad2) -> /power_r1
- J13 pad 2: unconnected-(J13-Pin_2-Pad2) -> /power_r2
- J14 pad 2: unconnected-(J14-Pin_2-Pad2) -> /power_r2
- J15 pad 2: unconnected-(J15-Pin_2-Pad2) -> /power_r2
- J16 pad 2: unconnected-(J16-Pin_2-Pad2) -> /power_r3
- J17 pad 2: unconnected-(J17-Pin_2-Pad2) -> /power_r3
- J18 pad 2: unconnected-(J18-Pin_2-Pad2) -> /power_r3
- J2 pad 2: unconnected-(J2-Pin_2-Pad2) -> /power_l1
- J3 pad 2: unconnected-(J3-Pin_2-Pad2) -> /power_l1
- J4 pad 2: unconnected-(J4-Pin_2-Pad2) -> /power_l2
- J5 pad 2: unconnected-(J5-Pin_2-Pad2) -> /power_l2
- J6 pad 2: unconnected-(J6-Pin_2-Pad2) -> /power_l2
- J7 pad 2: unconnected-(J7-Pin_2-Pad2) -> /power_l3
- J8 pad 2: unconnected-(J8-Pin_2-Pad2) -> /power_l3
- J9 pad 2: unconnected-(J9-Pin_2-Pad2) -> /power_l3
- U1 pad 1: unconnected-(U1-GPIO0-Pad1) -> /l1_j1
- U1 pad 10: /l1_j1 -> /l2_j2
- U1 pad 11: /l1_j2 -> /l2_j3
- U1 pad 12: /l1_j3 -> unconnected-(U1-GPIO9-Pad12)
- U1 pad 14: /l2_j1 -> unconnected-(U1-GPIO10-Pad14)
- U1 pad 15: /l2_j2 -> unconnected-(U1-GPIO11-Pad15)
- U1 pad 16: /l2_j3 -> unconnected-(U1-GPIO12-Pad16)
- U1 pad 2: unconnected-(U1-GPIO1-Pad2) -> /l1_j2
- U1 pad 39: unconnected-(U1-VSYS-Pad39) -> Net-(D1-K)
- U1 pad 4: unconnected-(U1-GPIO2-Pad4) -> /l1_j3
- U1 pad 9: unconnected-(U1-GPIO6-Pad9) -> /l2_j1
Routing:
- net /power: track 0.00 -> 190.6 mm
- net /power_r2: track 0.00 -> 60.5 mm
- net /power_l2: track 0.00 -> 38.5 mm
- net /r1_j1: track 0.00 -> 23.7 mm
- net /r1_j3: track 0.00 -> 23.4 mm
- net /r1_j2: track 0.00 -> 22.3 mm
- net /power_l3: track 0.00 -> 18.3 mm
- net /r2_j1: track 0.00 -> 18.0 mm
- net /power_r1: track 0.00 -> 17.8 mm
- net /r2_j2: track 0.00 -> 16.0 mm
- net /r2_j3: track 0.00 -> 14.9 mm
- net /power_l1: track 0.00 -> 14.6 mm
- net /power_r3: track 0.00 -> 14.4 mm
- net Net-(D1-A): track 0.00 -> 14.1 mm
- net Net-(D1-K): track 0.00 -> 9.52 mm
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- added copper zone on B.Cu, net GND
- added copper zone on F.Cu, net GND
Other:
- board size 109.5 x 113.5 mm -> 48 x 110 mm
- board text added: "GND"
- board text added: "Hexapod v2.1 (c) rookidroid.com Make Robotics Accessible and Fun for Everyone"
- board text added: "L1_J1"
- board text added: "L1_J2"
- board text added: "L1_J3"
- board text added: "L2_J1"
- board text added: "L2_J2"
- board text added: "L2_J3"
- board text added: "L3_J1"
- board text added: "L3_J2"
- board text added: "L3_J3"
- board text added: "POWER"
- board text added: "R1_J1"
- board text added: "R1_J2"
- board text added: "R1_J3"
- board text added: "R2_J1"
- board text added: "R2_J2"
- board text added: "R2_J3"
- board text added: "R3_J1"
- board text added: "R3_J2"
- board text added: "R3_J3"
- board text added: "USB"
