File: pcb/hexapod/hexapod.kicad_sch (KiCad schematic)
At the start: 19 parts, among them J1 Conn_01x03, J10 Conn_01x03, J11 Conn_01x03, J12 Conn_01x03, J13 Conn_01x03, J14 Conn_01x03, J15 Conn_01x03, J16 Conn_01x03, J17 Conn_01x03, J18 Conn_01x03, J2 Conn_01x03, J3 Conn_01x03, J4 Conn_01x03, J5 Conn_01x03, J6 Conn_01x03, J7 Conn_01x03, J8 Conn_01x03, J9 Conn_01x03, U1 Pico

Commit message: update
Parts:
- U1: footprint RPi_Pico:RPi_Pico_SMD_TH -> RPi_Pico_SMD_TH
Connections:
- net l2_j2: now reaches J5.1 (Pin_1)
- net l2_j2: now also U1.6 (GPIO4)
- net GND: now reaches J5.3 (Pin_3)
- net GND: now also J1.3 (Pin_3), J10.3 (Pin_3), J11.3 (Pin_3), J12.3 (Pin_3), J13.3 (Pin_3), J14.3 (Pin_3), J15.3 (Pin_3), J16.3 (Pin_3), J17.3 (Pin_3), J18.3 (Pin_3), J2.3 (Pin_3), J3.3 (Pin_3), J4.3 (Pin_3), J6.3 (Pin_3), J7.3 (Pin_3), J8.3 (Pin_3), J9.3 (Pin_3), U1.13 (GND), U1.18 (GND), U1.23 (GND), U1.28 (GND), U1.3 (GND), U1.33 (AGND), U1.38 (GND), U1.8 (GND)
- net r3_j1: now reaches J16.1 (Pin_1)
- net r3_j1: now also U1.24 (GPIO18)
- net r2_j3: now reaches J15.1 (Pin_1)
- net r2_j3: now also U1.25 (GPIO19)
- net l1_j1: now reaches U1.1 (GPIO0)
- net l1_j1: now also J1.1 (Pin_1)
- net l3_j2: now reaches U1.10 (GPIO7)
- net l3_j2: now also J8.1 (Pin_1)
- net l3_j3: now reaches U1.11 (GPIO8)
- net l3_j3: now also J9.1 (Pin_1)
- net l1_j2: now reaches U1.2 (GPIO1)
- net l1_j2: now also J2.1 (Pin_1)
- net r3_j3: now reaches U1.21 (GPIO16)
- net r3_j3: now also J18.1 (Pin_1)
- net r3_j2: now reaches U1.22 (GPIO17)
- net r3_j2: now also J17.1 (Pin_1)
- net r2_j2: now reaches U1.26 (GPIO20)
- net r2_j2: now also J14.1 (Pin_1)
- net r2_j1: now reaches U1.27 (GPIO21)
- net r2_j1: now also J13.1 (Pin_1)
- net r1_j3: now reaches U1.29 (GPIO22)
- net r1_j3: now also J12.1 (Pin_1)
- net r1_j2: now reaches U1.31 (GPIO26_ADC0)
- net r1_j2: now also J11.1 (Pin_1)
- net r1_j1: now reaches U1.32 (GPIO27_ADC1)
- net r1_j1: now also J10.1 (Pin_1)
- net l1_j3: now reaches U1.4 (GPIO2)
- net l1_j3: now also J3.1 (Pin_1)
- net l2_j1: now reaches U1.5 (GPIO3)
- net l2_j1: now also J4.1 (Pin_1)
- net l2_j3: now reaches U1.7 (GPIO5)
- net l2_j3: now also J6.1 (Pin_1)
- net l3_j1: now reaches U1.9 (GPIO6)
- net l3_j1: now also J7.1 (Pin_1)
Other:
- moved on the sheet: J1, J10, J11, J12, J13, J14, J15, J16, J17, J18, J2, J3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

Commit message: update
Connections:
- net l1_j1: now also U1.10 (GPIO7); no longer U1.1 (GPIO0)
- net l1_j2: now also U1.11 (GPIO8); no longer U1.2 (GPIO1)
- net l1_j3: now also U1.12 (GPIO9); no longer U1.4 (GPIO2)
- net l2_j1: now also U1.14 (GPIO10); no longer U1.5 (GPIO3)
- net l2_j2: now also U1.15 (GPIO11); no longer U1.6 (GPIO4)
- net l2_j3: now also U1.16 (GPIO12); no longer U1.7 (GPIO5)
- net l3_j1: now also U1.17 (GPIO13); no longer U1.9 (GPIO6)
- net l3_j2: now also U1.19 (GPIO14); no longer U1.10 (GPIO7)
- net l3_j3: now also U1.20 (GPIO15); no longer U1.11 (GPIO8)
Changed lines of the file:
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@@
+	(wire
+		(pts
+			(xy 129.54 125.73) (xy 135.89 125.73)
+		)
+		(stroke
+			(width 0)
+			(type default)
+		)
+	)
 	(wire
 		(pts
@@
 	(wire
 		(pts
+			(xy 129.54 133.35) (xy 135.89 133.35)
+		)
+		(stroke
+			(width 0)
+			(type default)
+		)
+	)
+	(wire
+		(pts
 			(xy 129.54 107.95) (xy 135.89 107.95)
 		)
@@
 	(wire
 		(pts
+			(xy 129.54 115.57) (xy 135.89 115.57)
+		)
+		(stroke
+			(width 0)
+			(type default)
+		)
+	)
+	(wire
+		(pts
+			(xy 129.54 135.89) (xy 135.89 135.89)
+		)
+		(stroke
+			(width 0)
+			(type default)
+		)
+	)
+	(wire
+		(pts
 			(xy 77.47 63.5) (xy 83.82 63.5)
 		)
@@
 	(wire
 		(pts
+			(xy 129.54 128.27) (xy 135.89 128.27)
+		)
+		(stroke
+			(width 0)
+			(type default)
+		)
+	)
+	(wire
+		(pts
 			(xy 171.45 133.35) (xy 177.8 133.35)
 		)
@@
 	(wire
 		(pts
+			(xy 129.54 120.65) (xy 135.89 120.65)
+		)
+		(stroke
+			(width 0)
+			(type default)
+		)
+	)
+	(wire
+		(pts
 			(xy 129.54 110.49) (xy 135.89 110.49)
 		)
@@
 		)
 	)
-	(label "l3_j1"
-		(at 129.54 107.95 0)
-		(fields_autoplaced yes)
-		(effects
-			(font
-				(size 1.27 1.27)
-			)
-			(justify left bottom)
-		)
-	)
-	(label "l1_j2"
-		(at 129.54 90.17 0)
-		(fields_autoplaced yes)
-		(effects
-			(font
-				(size 1.27 1.27)
-			)
-			(justify left bottom)
+	(wire
+		(pts
+			(xy 129.54 123.19) (xy 135.89 123.19)
+		)
+		(stroke
+			(width 0)
+			(type default)
 		)
 	)
@@
 		)
 	)
-	(label "l2_j1"
-		(at 129.54 97.79 0)
+	(label "l3_j3"
+		(at 129.54 135.89 0)
 		(fields_autoplaced yes)
 		(effects
@@
 		)
 	)
-	(label "l1_j3"
-		(at 129.54 95.25 0)
+	(label "l1_j2"
+		(at 129.54 113.03 0)
 		(fields_autoplaced yes)
 		(effects
@@
 		)
 	)
+	(label "l2_j3"
+		(at 129.54 125.73 0)
+		(fields_autoplaced yes)
+		(effects
+			(font
+				(size 1.27 1.27)
+			)
+			(justify left bottom)
+		)
+	)
 	(label "r1_j3"
 		(at 241.3 24.13 0)
@@
 		)
 	)
-	(label "l2_j2"
-		(at 129.54 100.33 0)
+	(label "l1_j1"
+		(at 129.54 110.49 0)
 		(fields_autoplaced yes)
 		(effects
@@
 		)
 	)
-	(label "l2_j3"
-		(at 129.54 102.87 0)
-		(fields_autoplaced yes)
-		(effects
-			(font
-				(size 1.27 1.27)
-			)
-			(justify left bottom)
-		)
-	)
 	(label "r1_j2"
 		(at 214.63 24.13 0)
@@
 		)
 	)
+	(label "l2_j2"
+		(at 129.54 123.19 0)
+		(fields_autoplaced yes)
+		(effects
+			(font
+				(size 1.27 1.27)
+			)
+			(justify left bottom)
+		)
+	)
 	(label "r3_j2"
 		(at 173.99 133.35 0)
@@
 		)
 	)
+	(label "l3_j2"
+		(at 129.54 133.35 0)
+		(fields_autoplaced yes)
+		(effects
+			(font
+				(size 1.27 1.27)
+			)
+			(justify left bottom)
+		)
+	)
 	(label "r3_j3"
 		(at 173.99 135.89 0)
@@
 		)
 	)
-	(label "l3_j2"
-		(at 129.54 110.49 0)
-		(fields_autoplaced yes)
-		(effects
-			(font
-				(size 1.27 1.27)
-			)
-			(justify left bottom)
-		)
-	)
 	(label "r1_j1"
 		(at 173.99 107.95 0)
@@
 		)
 	)
-	(label "l1_j1"
-		(at 129.54 87.63 0)
-		(fields_autoplaced yes)
-		(effects
-			(font
-				(size 1.27 1.27)
-			)
-			(justify left bottom)
-		)
-	)
 	(label "r3_j1"
 		(at 186.69 63.5 0)
@@
 		)
 	)
+	(label "l1_j3"
+		(at 129.54 115.57 0)
+		(fields_autoplaced yes)
+		(effects
+			(font
+				(size 1.27 1.27)
+			)
+			(justify left bottom)
+		)
+	)
 	(label "l3_j2"
 		(at 80.01 63.5 0)
@@
 		)
 	)
-	(label "l3_j3"
-		(at 129.54 113.03 0)
+	(label "l3_j1"
+		(at 129.54 128.27 0)
 		(fields_autoplaced yes)
 		(effects
@@
 		(fields_autoplaced yes)
 		(effects
+			(font
+				(size 1.27 1.27)
+			)
+			(justify left bottom)
+		)
+	)
+	(label "l2_j1"
+		(at 129.54 120.65 0)
+		(fields_autoplaced yes)
+		(effects

Commit message: pcb design
Parts:
- added D1: D_Schottky, Diode_THT:D_T-1_P10.16mm_Horizontal, symbol Device:D_Schottky
- added J19: Conn_01x02, TerminalBlock:TerminalBlock_MaiXu_MX126-5.0-02P_1x02_P5.00mm, symbol Connector_Generic:Conn_01x02
- added U2, U3, U4, U5, U6, U7, U8: ~, Hexapod_Library:Mini360, symbol Hexapod_Library:Mini360
- U1: footprint RPi_Pico_SMD_TH -> MCU_RaspberryPi_and_Boards:RPi_Pico_SMD_TH
Connections:
- net GND: now also J19.2 (Pin_2), U2.2 (-input), U2.4 (-output), U3.2 (-input), U3.4 (-output), U4.2 (-input), U4.4 (-output), U5.2 (-input), U5.4 (-output), U6.2 (-input), U6.4 (-output), U7.2 (-input), U7.4 (-output), U8.2 (-input), U8.4 (-output)
- net l1_j1: now also U1.1 (GPIO0); no longer U1.10 (GPIO7)
- net l1_j2: now also U1.2 (GPIO1); no longer U1.11 (GPIO8)
- net l1_j3: now also U1.4 (GPIO2); no longer U1.12 (GPIO9)
- net l2_j1: now also U1.9 (GPIO6); no longer U1.14 (GPIO10)
- net l2_j2: now also U1.10 (GPIO7); no longer U1.15 (GPIO11)
- net l2_j3: now also U1.11 (GPIO8); no longer U1.16 (GPIO12)
- net power_l2: now reaches J5.2 (Pin_2)
- net power_l2: now also J4.2 (Pin_2), J6.2 (Pin_2), U3.3 (+output)
- net power_r3: now reaches J16.2 (Pin_2)
- net power_r3: now also J17.2 (Pin_2), J18.2 (Pin_2), U7.3 (+output)
- net power_r2: now reaches J15.2 (Pin_2)
- net power_r2: now also J13.2 (Pin_2), J14.2 (Pin_2), U6.3 (+output)
- net at U1.39 (VSYS): now also D1.1 (K)
- net power_l1: now reaches J1.2 (Pin_2)
- net power_l1: now also J2.2 (Pin_2), J3.2 (Pin_2), U2.3 (+output)
- net power_l3: now reaches J9.2 (Pin_2)
- net power_l3: now also J7.2 (Pin_2), J8.2 (Pin_2), U4.3 (+output)
- net power_r1: now reaches J10.2 (Pin_2)
- net power_r1: now also J11.2 (Pin_2), J12.2 (Pin_2), U5.3 (+output)
- new net: D1.2 (A), U8.3 (+output)
- new net power: J19.1 (Pin_1), U2.1 (+input), U3.1 (+input), U4.1 (+input), U5.1 (+input), U6.1 (+input), U7.1 (+input), U8.1 (+input)

Commit message: fix pcb
Parts:
- removed U3, U4, U6, U7: ~, Hexapod_Library:Mini360, symbol Hexapod_Library:Mini360
- U2, U5: footprint Hexapod_Library:Mini360 -> Hexapod_Library:XL4005
Connections:
- net power_l2 is gone; now on net power_l1: J4.2 (Pin_2), J5.2 (Pin_2), J6.2 (Pin_2)
- net power_l3 is gone; now on net power_l1: J7.2 (Pin_2), J8.2 (Pin_2), J9.2 (Pin_2)
- net power_r2 is gone; now on net power_r1: J13.2 (Pin_2), J14.2 (Pin_2), J15.2 (Pin_2)
- net power_r3 is gone; now on net power_r1: J16.2 (Pin_2), J17.2 (Pin_2), J18.2 (Pin_2)
- net l2_j1: now also U1.7 (GPIO5); no longer U1.9 (GPIO6)
- net l2_j2: now also U1.9 (GPIO6); no longer U1.10 (GPIO7)
- net l2_j3: now also U1.10 (GPIO7); no longer U1.11 (GPIO8)
- net l3_j1: now also U1.12 (GPIO9); no longer U1.17 (GPIO13)
- net l3_j2: now also U1.16 (GPIO12); no longer U1.19 (GPIO14)
- net l3_j3: now also U1.17 (GPIO13); no longer U1.20 (GPIO15)

Commit message: update
Connections:
- net VSYS: now reaches D1.1 (K), U1.39 (VSYS)
Other:
- moved on the sheet: D1, J19, U1, U2, U5, U8
